File: MPPT/Eagle/MPPT_ArdProMini/MPPT_ArdProMini.brd (EAGLE design)
At the start: 102 x 82 mm, 28 parts, among them M2 ARDUINO-PRO-MINI-5.0V#APC, Q1 IRLZ44Z, Q2 IRLZ44Z, Q3 IRLZ44Z, U2 IR2104

Commit message: pin headers
Connections:
- new net N$9: JP1.6, M2.J7.3, M2.J7.3_LONG
- net GND: no longer JP1.6
Routing:
- net N$9: track 0.00 -> 55.7 mm
- net VCC: track 129.3 -> 141.0 mm
- net GND: track 303.2 -> 304.8 mm
