File: MPPT/Eagle/MPPT_LCD/MPPT_LCD.sch (EAGLE design)
At the start: 12 parts, among them IC1 MCP23017SP, U1 ARDUINOR3LONGHEADERATBOTTOM, X2 HD44780LCD

Commit message: pin headers
Parts:
- removed JP1: (no value), tmb_connectors:M06LONGPADS
- removed JP3: (no value), tmb_connectors:M08LONGPADS
- removed JP4: (no value), tmb_connectors:M10LONGPADS
- removed U1: ARDUINOR3LONGHEADERATBOTTOM, tmb_boards:ARDUINOR3LONGHEADERATBOTTOM
- JP2: device tmb_connectors:M08LONGPADS -> tmb_connectors:M06_MPPT_DATA
Connections:
- removed net N$1: JP4.7, U1.GND
- removed net N$13: JP3.4, U1.D3
- removed net N$14: JP1.3, U1.A3
- removed net N$15: JP1.4, U1.A2
- removed net N$16: JP1.5, U1.A1
- removed net N$17: JP1.6, U1.A0
- removed net N$18: JP2.1, U1.VIN
- removed net N$20: JP2.3, U1.GND2
- removed net N$22: JP2.5, U1.3V
- removed net N$23: JP2.6, U1./RESET
- removed net N$24: JP2.7, U1.IOREF
- removed net N$25: JP2.8, U1.RESERVED
- removed net N$26: JP3.1, U1.D0
- removed net N$27: JP3.2, U1.D1
- removed net N$28: JP3.3, U1.D2
- removed net N$29: JP3.5, U1.D4
- removed net N$30: JP3.6, U1.D5
- removed net N$31: JP3.7, U1.D6
- removed net N$32: JP3.8, U1.D7
- removed net N$33: JP4.1, U1.D8
- removed net N$34: JP4.2, U1.D9
- removed net N$35: JP4.3, U1.D10
- removed net N$36: JP4.4, U1.D11
- removed net N$37: JP4.5, U1.D12
- removed net N$38: JP4.6, U1.D13
- removed net N$40: JP4.8, U1.AREF
- removed net N$41: JP4.9, U1.SDA
- removed net N$42: JP4.10, U1.SCL
- net 5V: now also JP2.10; no longer JP2.4, U1.5V
- net GND: now also JP2.11; no longer JP2.2, U1.GND1
- net N$11: now also JP2.13; no longer JP1.2, U1.A4/SDA
- net N$12: now also JP2.12; no longer JP1.1, U1.A5/SCL
Other:
- note added: "ver 0.6"
- note removed: "ver 0.5"
Changed lines of the file:
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@@
 <part name="GND1" library="supply1" deviceset="GND" device=""/>
 <part name="GND5" library="supply1" deviceset="GND" device=""/>
-<part name="U1" library="tmb_boards" deviceset="ARDUINOR3" device="LONGHEADERATBOTTOM"/>
-<part name="JP1" library="tmb_connectors" deviceset="M06" device="LONGPADS"/>
-<part name="JP2" library="tmb_connectors" deviceset="M08" device="LONGPADS"/>
-<part name="JP3" library="tmb_connectors" deviceset="M08" device="LONGPADS"/>
-<part name="JP4" library="tmb_connectors" deviceset="M10" device="LONGPADS"/>
 <part name="R1" library="adafruit" deviceset="R-US_" device="0207/10" value="4.7K"/>
 <part name="R2" library="adafruit" deviceset="R-US_" device="0207/10" value="4.7K"/>
@@
 <part name="S2" library="SparkFun-Electromechanical" deviceset="SWITCH-SPDT" device="PTH"/>
 <part name="SUPPLY6" library="tmb_symbol" deviceset="5V" device=""/>
+<part name="JP2" library="tmb_connectors" deviceset="M06_MPPT_DATA" device=""/>
 </parts>
 <sheets>
 <sheet>
 <plain>
-<text x="193.04" y="154.94" size="1.778" layer="91">ver 0.5</text>
+<text x="193.04" y="154.94" size="1.778" layer="91">ver 0.6</text>
 </plain>
 <instances>
@@
 <instance part="GND1" gate="1" x="152.4" y="60.96" rot="MR0"/>
 <instance part="GND5" gate="1" x="205.74" y="121.92" rot="MR0"/>
-<instance part="U1" gate="G$1" x="50.8" y="116.84" rot="MR270"/>
-<instance part="JP1" gate="G$1" x="86.36" y="99.06" rot="MR0"/>
-<instance part="JP2" gate="G$1" x="86.36" y="119.38" rot="MR0"/>
-<instance part="JP3" gate="G$1" x="15.24" y="104.14"/>
-<instance part="JP4" gate="G$1" x="10.16" y="137.16"/>
 <instance part="R1" gate="G$1" x="106.68" y="106.68" rot="R90"/>
 <instance part="R2" gate="G$1" x="96.52" y="104.14" rot="R90"/>
 <instance part="TM1" gate="G$1" x="152.4" y="68.58"/>
-<instance part="GND4" gate="1" x="101.6" y="114.3" rot="MR0"/>
+<instance part="GND4" gate="1" x="96.52" y="88.9" rot="MR0"/>
 <instance part="X2" gate="G$1" x="208.28" y="86.36" rot="R90"/>
 <instance part="S1" gate="-1" x="154.94" y="127" rot="R90"/>
@@
 <instance part="S1" gate="-4" x="154.94" y="111.76" rot="R90"/>
 <instance part="GND6" gate="1" x="165.1" y="106.68" rot="MR0"/>
-<instance part="SUPPLY1" gate="G$1" x="96.52" y="119.38"/>
+<instance part="SUPPLY1" gate="G$1" x="88.9" y="83.82"/>
 <instance part="SUPPLY2" gate="G$1" x="96.52" y="109.22"/>
 <instance part="SUPPLY3" gate="G$1" x="106.68" y="111.76"/>
@@
 <instance part="S2" gate="1" x="182.88" y="101.6" rot="R180"/>
 <instance part="SUPPLY6" gate="G$1" x="172.72" y="104.14"/>
+<instance part="JP2" gate="G$1" x="71.12" y="81.28"/>
 </instances>
 <busses>
@@
 <pinref part="GND1" gate="1" pin="GND"/>
 <pinref part="TM1" gate="G$1" pin="A"/>
-</segment>
-<segment>
-<pinref part="U1" gate="G$1" pin="GND1"/>
-<pinref part="JP2" gate="G$1" pin="2"/>
-<pinref part="GND4" gate="1" pin="GND"/>
-<wire x1="101.6" y1="116.84" x2="93.98" y2="116.84" width="0.1524" layer="91"/>
-<wire x1="93.98" y1="116.84" x2="93.98" y2="114.3" width="0.1524" layer="91"/>
-<wire x1="93.98" y1="114.3" x2="81.28" y2="114.3" width="0.1524" layer="91"/>
 </segment>
 <segment>
@@
 <wire x1="165.1" y1="116.84" x2="160.02" y2="116.84" width="0.1524" layer="91"/>
 </segment>
+<segment>
+<pinref part="GND4" gate="1" pin="GND"/>
+<wire x1="81.28" y1="91.44" x2="96.52" y2="91.44" width="0.1524" layer="91"/>
+<pinref part="JP2" gate="G$1" pin="11"/>
+</segment>
 </net>
 <net name="N$2" class="0">
@@
 <net name="N$11" class="0">
 <segment>
-<pinref part="U1" gate="G$1" pin="A4/SDA"/>
-<pinref part="JP1" gate="G$1" pin="2"/>
 <pinref part="IC1" gate="G$1" pin="SDA"/>
 <wire x1="81.28" y1="96.52" x2="96.52" y2="96.52" width="0.1524" layer="91"/>
@@
 <wire x1="96.52" y1="96.52" x2="116.84" y2="96.52" width="0.1524" layer="91"/>
 <wire x1="96.52" y1="96.52" x2="96.52" y2="99.06" width="0.1524" layer="91"/>
+<pinref part="JP2" gate="G$1" pin="13"/>
 </segment>
 </net>
 <net name="N$12" class="0">
 <segment>
-<pinref part="U1" gate="G$1" pin="A5/SCL"/>
-<pinref part="JP1" gate="G$1" pin="1"/>
 <pinref part="IC1" gate="G$1" pin="SCL"/>
 <wire x1="116.84" y1="99.06" x2="106.68" y2="99.06" width="0.1524" layer="91"/>
@@
 <pinref part="R1" gate="G$1" pin="1"/>
 <wire x1="106.68" y1="99.06" x2="106.68" y2="101.6" width="0.1524" layer="91"/>
-</segment>
-</net>
-<net name="N$13" class="0">
-<segment>
-<pinref part="U1" gate="G$1" pin="D3"/>
-<pinref part="JP3" gate="G$1" pin="4"/>
-</segment>
-</net>
-<net name="N$14" class="0">
-<segment>
-<pinref part="U1" gate="G$1" pin="A3"/>
-<pinref part="JP1" gate="G$1" pin="3"/>
-</segment>
-</net>
-<net name="N$15" class="0">
-<segment>
-<pinref part="U1" gate="G$1" pin="A2"/>
-<pinref part="JP1" gate="G$1" pin="4"/>
-</segment>
-</net>
-<net name="N$16" class="0">
-<segment>
-<pinref part="U1" gate="G$1" pin="A1"/>
-<pinref part="JP1" gate="G$1" pin="5"/>
-</segment>
-</net>
-<net name="N$17" class="0">
-<segment>
-<pinref part="U1" gate="G$1" pin="A0"/>
-<pinref part="JP1" gate="G$1" pin="6"/>
-</segment>
-</net>
-<net name="N$18" class="0">
-<segment>
-<pinref part="U1" gate="G$1" pin="VIN"/>
-<pinref part="JP2" gate="G$1" pin="1"/>
-</segment>
-</net>
-<net name="N$20" class="0">
-<segment>
-<pinref part="U1" gate="G$1" pin="GND2"/>
-<pinref part="JP2" gate="G$1" pin="3"/>
-</segment>
-</net>
-<net name="N$22" class="0">
-<segment>
-<pinref part="U1" gate="G$1" pin="3V"/>
-<pinref part="JP2" gate="G$1" pin="5"/>
-</segment>
-</net>
-<net name="N$23" class="0">
-<segment>
-<pinref part="U1" gate="G$1" pin="/RESET"/>
-<pinref part="JP2" gate="G$1" pin="6"/>
-</segment>
-</net>
-<net name="N$24" class="0">
-<segment>
-<pinref part="U1" gate="G$1" pin="IOREF"/>
-<pinref part="JP2" gate="G$1" pin="7"/>
-</segment>
-</net>
-<net name="N$25" class="0">
-<segment>
-<pinref part="U1" gate="G$1" pin="RESERVED"/>
-<pinref part="JP2" gate="G$1" pin="8"/>
-</segment>
-</net>
-<net name="N$26" class="0">
-<segment>
-<pinref part="U1" gate="G$1" pin="D0"/>
-<pinref part="JP3" gate="G$1" pin="1"/>
-</segment>
-</net>
-<net name="N$27" class="0">
-<segment>
-<pinref part="U1" gate="G$1" pin="D1"/>
-<pinref part="JP3" gate="G$1" pin="2"/>
-</segment>
-</net>
-<net name="N$28" class="0">
-<segment>
-<pinref part="U1" gate="G$1" pin="D2"/>
-<pinref part="JP3" gate="G$1" pin="3"/>
-</segment>
-</net>
-<net name="N$29" class="0">
-<segment>
-<pinref part="U1" gate="G$1" pin="D4"/>
-<pinref part="JP3" gate="G$1" pin="5"/>
-</segment>
-</net>
-<net name="N$30" class="0">
-<segment>
-<pinref part="U1" gate="G$1" pin="D5"/>
-<pinref part="JP3" gate="G$1" pin="6"/>
-</segment>
-</net>
-<net name="N$31" class="0">
-<segment>
-<pinref part="U1" gate="G$1" pin="D6"/>
-<pinref part="JP3" gate="G$1" pin="7"/>
-</segment>
-</net>
-<net name="N$32" class="0">
-<segment>
-<pinref part="U1" gate="G$1" pin="D7"/>
-<pinref part="JP3" gate="G$1" pin="8"/>
-</segment>
-</net>
-<net name="N$33" class="0">
-<segment>
-<pinref part="U1" gate="G$1" pin="D8"/>
-<pinref part="JP4" gate="G$1" pin="1"/>
-</segment>
-</net>
-<net name="N$34" class="0">
-<segment>
-<pinref part="U1" gate="G$1" pin="D9"/>
-<pinref part="JP4" gate="G$1" pin="2"/>
-</segment>
-</net>
-<net name="N$35" class="0">
-<segment>
-<pinref part="U1" gate="G$1" pin="D10"/>
-<pinref part="JP4" gate="G$1" pin="3"/>
-</segment>
-</net>
-<net name="N$36" class="0">
-<segment>
-<pinref part="U1" gate="G$1" pin="D11"/>
-<pinref part="JP4" gate="G$1" pin="4"/>
-</segment>
-</net>
-<net name="N$37" class="0">
-<segment>
-<pinref part="U1" gate="G$1" pin="D12"/>
-<pinref part="JP4" gate="G$1" pin="5"/>
-</segment>
-</net>
-<net name="N$38" class="0">
-<segment>
-<pinref part="U1" gate="G$1" pin="D13"/>
-<pinref part="JP4" gate="G$1" pin="6"/>
-</segment>
-</net>
-<net name="N$40" class="0">
-<segment>
-<pinref part="U1" gate="G$1" pin="AREF"/>
-<pinref part="JP4" gate="G$1" pin="8"/>
-</segment>
-</net>
-<net name="N$41" class="0">
-<segment>
-<pinref part="U1" gate="G$1" pin="SDA"/>
-<pinref part="JP4" gate="G$1" pin="9"/>
-</segment>
-</net>
-<net name="N$42" class="0">
-<segment>
-<pinref part="U1" gate="G$1" pin="SCL"/>
-<pinref part="JP4" gate="G$1" pin="10"/>
-</segment>
-</net>
-<net name="N$1" class="0">
-<segment>
-<pinref part="U1" gate="G$1" pin="GND"/>
-<pinref part="JP4" gate="G$1" pin="7"/>
+<pinref part="JP2" gate="G$1" pin="12"/>
 </segment>
 </net>
@@
 </net>
 <net name="5V" class="0">
-<segment>
-<pinref part="U1" gate="G$1" pin="5V"/>
-<pinref part="JP2" gate="G$1" pin="4"/>
-<wire x1="96.52" y1="119.38" x2="81.28" y2="119.38" width="0.1524" layer="91"/>
-<pinref part="SUPPLY1" gate="G$1" pin="5V"/>
-</segment>
 <segment>
 <pinref part="R2" gate="G$1" pin="2"/>
@@
 <wire x1="177.8" y1="104.14" x2="172.72" y2="104.14" width="0.1524" layer="91"/>
 </segment>
-</net>
+<segment>
+<pinref part="SUPPLY1" gate="G$1" pin="5V"/>
+<wire x1="88.9" y1="83.82" x2="83.82" y2="83.82" width="0.1524" layer="91"/>
+<wire x1="83.82" y1="83.82" x2="83.82" y2="88.9" width="0.1524" layer="91"/>
+<wire x1="83.82" y1="88.9" x2="81.28" y2="88.9" width="0.1524" layer="91"/>
+<pinref part="JP2" gate="G$1" pin="10"/>
+</segment>
+</net>
