File: MPPT/Eagle/MPPT_power/MPPT_power.brd (EAGLE design)
At the start: 102 x 82 mm, 22 parts, among them K3 5V, T2 BC337, X1 SWITCHDOC_INA3221

Commit message: pin headers
Parts:
- removed K3: 5V, tmb_relay:G5V-2
- removed R3, R4: 0.1, tmb_resistor:0204/7
- removed S1: (no value), SparkFun-Electromechanical:SWITCH-SPDT
- added K1: HX2-5V, tmb_relay:HX
- added R2, R6: 0.1, tmb_resistor:0204/7_PHAT_PAD
- added S2: (no value), tmb_switch:SWITCH-SPDT_0.15_INCH
Connections:
- net GND: now also K1.12; no longer JP2.6, K3.16
- net N$1: now also K1.9, R2.2; no longer K3.13, R4.2
- net N$13: now also K1.1; no longer K3.1
- net N$15: now also R2.1; no longer R4.1
- net N$16: now also R6.1; no longer R3.1
- net N$5: now also S2.2; no longer S1.2
- net N$6: now also R6.2; no longer R3.2
- net N$9: now also K1.8, S2.1; no longer K3.9, S1.1
Routing:
- net N$16: track 51.8 -> 33.0 mm
- net GND: track 330.8 -> 320.3 mm
- net N$6: track 25.7 -> 34.8 mm
- net N$9: track 29.5 -> 34.8 mm
- net N$13: track 9.80 -> 12.9 mm
- net N$5: track 26.2 -> 23.6 mm
- net 5V: track 139.9 -> 140.8 mm
