File: MPPT/Eagle/MPPT_power/MPPT_power.sch (EAGLE design)
At the start: 22 parts, among them K3 5V, T2 BC337, X1 SWITCHDOC_INA3221

Commit message: pin headers
Parts:
- removed K3: 5V, tmb_relay:G5V-2
- removed R3, R4: 0.1, tmb_resistor:R-US_0204/7
- removed S1: (no value), SparkFun-Electromechanical:SWITCH-SPDTPTH
- added K1: HX2-5V, tmb_relay:HX2-5V
- added R2, R6: 0.1, tmb_resistor:R-US_
- added S2: (no value), tmb_switch:SWITCH-SPDT
Connections:
- net GND: now also K11.2; no longer JP2.6, K3A.2
- net N$1: now also K13.P, R2.2; no longer K32.P, R4.2
- net N$13: now also K11.1; no longer K3A.1
- net N$15: now also R2.1; no longer R4.1
- net N$16: now also R6.1; no longer R3.1
- net N$5: now also S2.P; no longer S1.P
- net N$6: now also R6.2; no longer R3.2
- net N$9: now also K13.S, S2.O; no longer K32.S, S1.O
Other:
- note added: "rev 0.6"
- note removed: "rev 0.5"
Changed lines of the file:
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@@
 </classes>
 <parts>
-<part name="S1" library="SparkFun-Electromechanical" deviceset="SWITCH-SPDT" device="PTH"/>
 <part name="GND3" library="SparkFun-Aesthetics" deviceset="GND" device=""/>
 <part name="GND4" library="SparkFun-Aesthetics" deviceset="GND" device=""/>
-<part name="K3" library="tmb_relay" deviceset="G5V-2" device="" value="5V"/>
 <part name="GND9" library="SparkFun-Aesthetics" deviceset="GND" device=""/>
 <part name="GND14" library="SparkFun-Aesthetics" deviceset="GND" device=""/>
@@
 <part name="SUPPLY4" library="SparkFun-Aesthetics" deviceset="5V" device=""/>
 <part name="GND8" library="SparkFun-Aesthetics" deviceset="GND" device=""/>
-<part name="R3" library="tmb_resistor" deviceset="R-US_" device="0204/7" value="0.1"/>
-<part name="R4" library="tmb_resistor" deviceset="R-US_" device="0204/7" value="0.1"/>
 <part name="SUPPLY3" library="SparkFun-Aesthetics" deviceset="5V" device=""/>
 <part name="GND5" library="SparkFun-Aesthetics" deviceset="GND" device=""/>
@@
 <part name="R5" library="tmb_resistor" deviceset="R-US_" device="0204/7" value="10K"/>
 <part name="GND12" library="SparkFun-Aesthetics" deviceset="GND" device=""/>
+<part name="K1" library="tmb_relay" deviceset="HX2-*" device="" technology="5V"/>
+<part name="S2" library="tmb_switch" deviceset="SWITCH-SPDT" device=""/>
+<part name="R2" library="tmb_resistor" deviceset="R-US_" device="" value="0.1"/>
+<part name="R6" library="tmb_resistor" deviceset="R-US_" device="" value="0.1"/>
 </parts>
 <sheets>
 <sheet>
 <plain>
-<text x="180.34" y="119.38" size="1.778" layer="91">rev 0.5</text>
+<text x="180.34" y="119.38" size="1.778" layer="91">rev 0.6</text>
 </plain>
 <instances>
-<instance part="S1" gate="1" x="20.32" y="124.46"/>
 <instance part="GND3" gate="1" x="15.24" y="96.52"/>
 <instance part="GND4" gate="1" x="15.24" y="38.1" rot="MR0"/>
-<instance part="K3" gate="A" x="121.92" y="121.92"/>
-<instance part="K3" gate="2" x="33.02" y="121.92"/>
 <instance part="GND9" gate="1" x="121.92" y="111.76"/>
 <instance part="GND14" gate="1" x="101.6" y="111.76"/>
@@
 <instance part="GND2" gate="1" x="40.64" y="96.52"/>
 <instance part="U$3" gate="G$1" x="147.32" y="73.66"/>
-<instance part="GND1" gate="1" x="22.86" y="68.58"/>
+<instance part="GND1" gate="1" x="22.86" y="66.04"/>
 <instance part="X1" gate="G$2" x="104.14" y="55.88" rot="MR0"/>
 <instance part="SUPPLY4" gate="G$1" x="121.92" y="58.42" rot="MR0"/>
 <instance part="GND8" gate="1" x="114.3" y="58.42" rot="MR0"/>
-<instance part="R3" gate="G$1" x="30.48" y="60.96" rot="MR180"/>
-<instance part="R4" gate="G$1" x="40.64" y="66.04" rot="MR180"/>
 <instance part="SUPPLY3" gate="G$1" x="30.48" y="81.28" rot="MR0"/>
 <instance part="GND5" gate="1" x="22.86" y="81.28" rot="MR0"/>
@@
 <instance part="R5" gate="G$1" x="-2.54" y="58.42" rot="R270"/>
 <instance part="GND12" gate="1" x="-2.54" y="48.26"/>
+<instance part="K1" gate="1" x="121.92" y="121.92"/>
+<instance part="K1" gate="2" x="162.56" y="106.68"/>
+<instance part="K1" gate="3" x="33.02" y="121.92"/>
+<instance part="S2" gate="1" x="20.32" y="124.46"/>
+<instance part="R2" gate="G$1" x="40.64" y="66.04"/>
+<instance part="R6" gate="G$1" x="30.48" y="60.96"/>
 </instances>
 <busses>
@@
 <pinref part="D1" gate="1" pin="A"/>
 <wire x1="111.76" y1="119.38" x2="111.76" y2="114.3" width="0.1524" layer="91"/>
-<pinref part="K3" gate="A" pin="2"/>
+<pinref part="K1" gate="1" pin="2"/>
 </segment>
 <segment>
@@
 </segment>
 <segment>
-<pinref part="GND1" gate="1" pin="GND"/>
-<wire x1="22.86" y1="71.12" x2="15.24" y2="71.12" width="0.1524" layer="91"/>
-<pinref part="JP2" gate="G$1" pin="6"/>
-<pinref part="JP2" gate="G$1" pin="5"/>
-<wire x1="15.24" y1="71.12" x2="15.24" y2="68.58" width="0.1524" layer="91"/>
-</segment>
-<segment>
 <pinref part="GND5" gate="1" pin="GND"/>
 <wire x1="22.86" y1="83.82" x2="15.24" y2="83.82" width="0.1524" layer="91"/>
@@
 <pinref part="GND12" gate="1" pin="GND"/>
 <wire x1="-2.54" y1="53.34" x2="-2.54" y2="50.8" width="0.1524" layer="91"/>
+</segment>
+<segment>
+<pinref part="JP2" gate="G$1" pin="5"/>
+<pinref part="GND1" gate="1" pin="GND"/>
+<wire x1="15.24" y1="68.58" x2="22.86" y2="68.58" width="0.1524" layer="91"/>
 </segment>
 </net>
@@
 <pinref part="D1" gate="1" pin="C"/>
 <wire x1="111.76" y1="129.54" x2="111.76" y2="124.46" width="0.1524" layer="91"/>
-<pinref part="K3" gate="A" pin="1"/>
+<pinref part="K1" gate="1" pin="1"/>
 </segment>
 </net>
@@
 <net name="N$9" class="0">
 <segment>
-<pinref part="S1" gate="1" pin="O"/>
 <wire x1="27.94" y1="127" x2="25.4" y2="127" width="0.1524" layer="91"/>
-<pinref part="K3" gate="2" pin="S"/>
 <pinref part="START" gate="1" pin="P1"/>
 <wire x1="30.48" y1="132.08" x2="27.94" y2="132.08" width="0.1524" layer="91"/>
 <wire x1="27.94" y1="132.08" x2="27.94" y2="127" width="0.1524" layer="91"/>
+<pinref part="K1" gate="3" pin="S"/>
+<junction x="27.94" y="127"/>
+<pinref part="S2" gate="1" pin="O"/>
 </segment>
 </net>
@@
 <net name="N$5" class="0">
 <segment>
-<pinref part="S1" gate="1" pin="P"/>
 <pinref part="U$7" gate="G$1" pin="2"/>
 <wire x1="17.78" y1="124.46" x2="15.24" y2="124.46" width="0.1524" layer="91"/>
+<pinref part="S2" gate="1" pin="P"/>
 </segment>
 </net>
 <net name="N$15" class="0">
 <segment>
-<pinref part="R4" gate="G$1" pin="1"/>
 <wire x1="35.56" y1="66.04" x2="33.02" y2="66.04" width="0.1524" layer="91"/>
 <wire x1="33.02" y1="66.04" x2="33.02" y2="63.5" width="0.1524" layer="91"/>
@@
 <pinref part="D3" gate="1" pin="A"/>
 <wire x1="132.08" y1="99.06" x2="132.08" y2="93.98" width="0.1524" layer="91"/>
+<pinref part="R2" gate="G$1" pin="1"/>
 </segment>
 </net>
 <net name="N$16" class="0">
 <segment>
-<pinref part="R3" gate="G$1" pin="1"/>
 <wire x1="25.4" y1="60.96" x2="22.86" y2="60.96" width="0.1524" layer="91"/>
 <wire x1="22.86" y1="60.96" x2="22.86" y2="58.42" width="0.1524" layer="91"/>
@@
 <pinref part="JP2" gate="G$1" pin="2"/>
 <wire x1="15.24" y1="60.96" x2="15.24" y2="58.42" width="0.1524" layer="91"/>
+<pinref part="R6" gate="G$1" pin="1"/>
 </segment>
 </net>
@@
 <segment>
 <pinref part="START" gate="1" pin="S1"/>
-<pinref part="K3" gate="2" pin="P"/>
 <wire x1="33.02" y1="119.38" x2="40.64" y2="119.38" width="0.1524" layer="91"/>
 <pinref part="U$13" gate="G$1" pin="2"/>
@@
 <pinref part="R1" gate="G$1" pin="1"/>
 <junction x="40.64" y="119.38"/>
-<pinref part="R4" gate="G$1" pin="2"/>
 <pinref part="X1" gate="G$2" pin="IN+2"/>
 <wire x1="45.72" y1="66.04" x2="48.26" y2="66.04" width="0.1524" layer="91"/>
 <wire x1="48.26" y1="66.04" x2="76.2" y2="66.04" width="0.1524" layer="91"/>
 <wire x1="48.26" y1="119.38" x2="48.26" y2="66.04" width="0.1524" layer="91"/>
+<pinref part="K1" gate="3" pin="P"/>
+<pinref part="R2" gate="G$1" pin="2"/>
 </segment>
 </net>
@@
 <segment>
 <pinref part="X1" gate="G$2" pin="IN+3"/>
-<pinref part="R3" gate="G$1" pin="2"/>
 <wire x1="35.56" y1="60.96" x2="38.1" y2="60.96" width="0.1524" layer="91"/>
 <pinref part="U$1" gate="G$1" pin="2"/>
@@
 <wire x1="15.24" y1="45.72" x2="38.1" y2="45.72" width="0.1524" layer="91"/>
 <wire x1="38.1" y1="60.96" x2="38.1" y2="45.72" width="0.1524" layer="91"/>
-</segment>
-</net>
+<pinref part="R6" gate="G$1" pin="2"/>
+</segment>
+</net>
